File: hardware/ADXL377 Breakout.sch (EAGLE design)
At the start: 13 parts, among them U1 ADXL377

Commit message: Added 4 mounting holes and modified silk, ready for protos
Parts:
- added STANDOFF2, STANDOFF3, STANDOFF4: STAND-OFF, SparkFun-Electromechanical:STAND-OFF
- renumbered LOGO3 to LOGO5
Changed lines of the file:
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@@
 <part name="LOGO1" library="SparkFun-Aesthetics" deviceset="SFE_LOGO_FLAME" device=".1_INCH"/>
 <part name="LOGO2" library="SparkFun-Aesthetics" deviceset="OSHW-LOGO" device="S"/>
-<part name="LOGO3" library="SparkFun-Aesthetics" deviceset="SFE_LOGO_NAME_FLAME" device=".1_INCH"/>
+<part name="LOGO5" library="SparkFun-Aesthetics" deviceset="SFE_LOGO_NAME_FLAME" device=".1_INCH"/>
+<part name="STANDOFF2" library="SparkFun-Electromechanical" deviceset="STAND-OFF" device=""/>
+<part name="STANDOFF3" library="SparkFun-Electromechanical" deviceset="STAND-OFF" device=""/>
+<part name="STANDOFF4" library="SparkFun-Electromechanical" deviceset="STAND-OFF" device=""/>
 </parts>
 <sheets>
@@
 <instance part="LOGO1" gate="G$1" x="236.22" y="38.1"/>
 <instance part="LOGO2" gate="G$1" x="220.98" y="45.72"/>
-<instance part="LOGO3" gate="G$1" x="88.9" y="0"/>
+<instance part="LOGO5" gate="G$1" x="88.9" y="0"/>
+<instance part="STANDOFF2" gate="G$1" x="238.76" y="30.48"/>
+<instance part="STANDOFF3" gate="G$1" x="233.68" y="30.48"/>
+<instance part="STANDOFF4" gate="G$1" x="228.6" y="30.48"/>
 </instances>
 <busses>

Commit message: v10 ready for review
Other:
- note added: "v10"
- note removed: "v01"
Changed lines of the file:
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@@
 <plain>
 <text x="149.86" y="7.62" size="2.54" layer="94">Jordan McConnell</text>
-<text x="238.76" y="7.62" size="2.54" layer="94">v01</text>
+<text x="238.76" y="7.62" size="2.54" layer="94">v10</text>
 </plain>
 <instances>

Commit message: v10, ready for reds
Parts:
- removed LOGO5: SFE_LOGO_NAME_FLAME.1_INCH, SparkFun-Aesthetics:SFE_LOGO_NAME_FLAME.1_INCH
Changed lines of the file:
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@@
 <part name="LOGO1" library="SparkFun-Aesthetics" deviceset="SFE_LOGO_FLAME" device=".1_INCH"/>
 <part name="LOGO2" library="SparkFun-Aesthetics" deviceset="OSHW-LOGO" device="S"/>
-<part name="LOGO5" library="SparkFun-Aesthetics" deviceset="SFE_LOGO_NAME_FLAME" device=".1_INCH"/>
 <part name="STANDOFF2" library="SparkFun-Electromechanical" deviceset="STAND-OFF" device=""/>
 <part name="STANDOFF3" library="SparkFun-Electromechanical" deviceset="STAND-OFF" device=""/>
@@
 <instance part="LOGO1" gate="G$1" x="236.22" y="38.1"/>
 <instance part="LOGO2" gate="G$1" x="220.98" y="45.72"/>
-<instance part="LOGO5" gate="G$1" x="88.9" y="0"/>
 <instance part="STANDOFF2" gate="G$1" x="238.76" y="30.48"/>
 <instance part="STANDOFF3" gate="G$1" x="233.68" y="30.48"/>
